File: actuator/10001/10001.kicad_sch (KiCad schematic)
At the start: 0 parts

Commit message: 10001 schematic work
Other:
- added sheet Buck Converter (buck.kicad_sch)
- company: Jay Maybe -> James May
Changed lines of the file:
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@@
 		(date "2026-07-22")
 		(rev "001")
-		(company "Jay Maybe")
-	)
-	(sheet
-		(at 50.8 140.97)
-		(size 45.72 31.75)
+		(company "James May")
+	)
+	(sheet
+		(at 38.1 50.8)
+		(size 38.1 38.1)
+		(exclude_from_sim no)
+		(in_bom yes)
+		(on_board yes)
+		(dnp no)
+		(fields_autoplaced yes)
+		(stroke
+			(width 0.1524)
+			(type solid)
+		)
+		(fill
+			(color 0 0 0 0)
+		)
+		(property "Sheetname" "Buck Converter"
+			(at 38.1 50.0884 0)
+			(show_name no)
+			(do_not_autoplace no)
+			(effects
+				(font
+					(size 1.27 1.27)
+				)
+				(justify left bottom)
+			)
+		)
+		(property "Sheetfile" "buck.kicad_sch"
+			(at 38.1 89.4846 0)
+			(show_name no)
+			(do_not_autoplace no)
+			(effects
+				(font
+					(size 1.27 1.27)
+				)
+				(justify left top)
+			)
+		)
+		(instances
+			(project "10001"
+				(path "/74a9143e-df50-4944-bff2-a4302f33bdee"
+					(page "6")
+				)
+			)
+		)
+	)
+	(sheet
+		(at 165.1 50.8)
+		(size 38.1 38.1)
 		(exclude_from_sim no)
 		(in_bom yes)
@@
 		)
 		(property "Sheetname" "Motor Driver"
-			(at 50.8 140.2584 0)
+			(at 165.1 50.0884 0)
 			(show_name no)
 			(do_not_autoplace no)
@@
 		)
 		(property "Sheetfile" "motordriver.kicad_sch"
-			(at 50.8 173.3046 0)
+			(at 165.1 89.4846 0)
 			(show_name no)
 			(do_not_autoplace no)
@@
 	)
 	(sheet
-		(at 151.13 92.71)
-		(size 41.91 39.37)
+		(at 165.1 101.6)
+		(size 38.1 38.1)
 		(exclude_from_sim no)
 		(in_bom yes)
@@
 		)
 		(property "Sheetname" "Encoder"
-			(at 151.13 91.9984 0)
+			(at 165.1 100.8884 0)
 			(show_name no)
 			(do_not_autoplace no)
@@
 		)
 		(property "Sheetfile" "encoder.kicad_sch"
-			(at 151.13 132.6646 0)
+			(at 165.1 140.2846 0)
 			(show_name no)
 			(do_not_autoplace no)
@@
 	)
 	(sheet
-		(at 143.51 59.69)
-		(size 27.94 13.97)
+		(at 38.1 101.6)
+		(size 25.4 25.4)
 		(exclude_from_sim no)
 		(in_bom yes)
@@
 		)
 		(property "Sheetname" "LDO"
-			(at 143.51 58.9784 0)
+			(at 38.1 100.8884 0)
 			(show_name no)
 			(do_not_autoplace no)
@@
 		)
 		(property "Sheetfile" "ldo.kicad_sch"
-			(at 143.51 74.2446 0)
+			(at 38.1 127.5846 0)
 			(show_name no)
 			(do_not_autoplace no)
@@
 	)
 	(sheet
-		(at 67.31 66.04)
-		(size 36.83 38.1)
+		(at 101.6 50.8)
+		(size 38.1 38.1)
 		(exclude_from_sim no)
 		(in_bom yes)
@@
 		)
 		(property "Sheetname" "Microcontroller"
-			(at 67.31 65.3284 0)
+			(at 101.6 50.0884 0)
 			(show_name no)
 			(do_not_autoplace no)
@@
 		)
 		(property "Sheetfile" "micro.kicad_sch"
-			(at 67.31 104.7246 0)
-			(show_name no)
-			(do_not_autoplace no)
+			(at 101.6 89.4846 0)
+			(show_name no)
+			(do_not_autoplace no)
