File: actuator/10001/ldo.kicad_sch (KiCad schematic)
At the start: 0 parts

Commit message: 10001 schematic work
Other:
- company: Jay Maybe -> James May
Changed lines of the file:
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@@
 		(date "2026-07-22")
 		(rev "001")
-		(company "Jay Maybe")
+		(company "James May")
 	)
 )
