File: actuator/10001/buck.kicad_sch (KiCad schematic)
At the start: 33 parts, among them Q1 DMN6140L, Q2 DMN6140L, U4 LM5117

Commit message: checkpoint
Parts:
- C10: renamed from C4; footprint (none) -> Capacitor_SMD:C_0805_2012Metric
- C11: renamed from C10; footprint (none) -> Capacitor_SMD:C_0805_2012Metric
- C12: renamed from C11; footprint (none) -> Capacitor_SMD:C_0805_2012Metric
- C13: footprint (none) -> Capacitor_SMD:C_0805_2012Metric
- C14: renamed from C12; footprint (none) -> Capacitor_SMD:C_0805_2012Metric
- C15: renamed from C8; footprint (none) -> Capacitor_SMD:C_0805_2012Metric
- C16: renamed from C5; footprint (none) -> Capacitor_SMD:C_0805_2012Metric
- C17: renamed from C15; footprint (none) -> Capacitor_SMD:C_0805_2012Metric
- C18: renamed from C6; footprint (none) -> Capacitor_SMD:C_0805_2012Metric
- C19: renamed from C14; footprint (none) -> Capacitor_SMD:C_0805_2012Metric
- C20: renamed from C7; footprint (none) -> Capacitor_SMD:C_0805_2012Metric
- C7: renamed from C3; footprint (none) -> Capacitor_SMD:C_0805_2012Metric
- C8: renamed from C1; footprint (none) -> Capacitor_SMD:C_0805_2012Metric
- C9: renamed from C2; footprint (none) -> Capacitor_SMD:C_0805_2012Metric
- R10: renamed from R13; footprint (none) -> Resistor_SMD:R_0805_2012Metric
- R11: renamed from R7; footprint (none) -> Resistor_SMD:R_0805_2012Metric
- R12: renamed from R9; footprint (none) -> Resistor_SMD:R_0805_2012Metric
- R13: renamed from R14; footprint (none) -> Resistor_SMD:R_0805_2012Metric
- R14: renamed from R8; footprint (none) -> Resistor_SMD:R_0805_2012Metric
- R15: renamed from R10; footprint (none) -> Resistor_SMD:R_0805_2012Metric
- R4: renamed from R3; footprint (none) -> Resistor_SMD:R_0805_2012Metric
- R5: renamed from R4; footprint (none) -> Resistor_SMD:R_0805_2012Metric
- R6: renamed from R5; footprint (none) -> Resistor_SMD:R_0805_2012Metric
- R7: renamed from R6; footprint (none) -> Resistor_SMD:R_0805_2012Metric
- R8: renamed from R11; footprint (none) -> Resistor_SMD:R_0805_2012Metric
- R9: renamed from R12; footprint (none) -> Resistor_SMD:R_0805_2012Metric
