File: actuator/10001/encoder.kicad_sch (KiCad schematic)
At the start: 5 parts

Commit message: 10001 schematic work
Parts:
- U1: value (none) -> LDC0851
Other:
- company: Jay Maybe -> James May
Changed lines of the file:
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@@
 		(date "2026-07-22")
 		(rev "001")
-		(company "Jay Maybe")
+		(company "James May")
 	)
 	(junction
@@
 		(in_pos_files yes)
 		(dnp no)
-		(fields_autoplaced yes)
 		(property "Reference" "U1"
-			(at 144.3833 71.12 0)
+			(at 146.05 69.85 0)
 			(show_name no)
 			(do_not_autoplace no)
@@
 			)
 		)
-		(property "Value" ""
-			(at 142.24 73.66 0)
-			(show_name no)
-			(do_not_autoplace no)
+		(property "Value" "LDC0851"
+			(at 147.32 72.39 0)
+			(show_name no)
+			(do_not_autoplace no)

Commit message: checkpoint
Parts:
- renumbered R1 to R3, U1 to U3
Changed lines of the file:
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@@
 		(dnp no)
 		(fields_autoplaced yes)
-		(property "Reference" "R1"
+		(property "Reference" "R3"
 			(at 116.84 116.8399 0)
 			(show_name no)
@@
 			(project "10001"
 				(path "/74a9143e-df50-4944-bff2-a4302f33bdee/58f0d544-aaa2-42db-8316-207d7dca1f4a"
-					(reference "R1")
+					(reference "R3")
 					(unit 1)
 				)
@@
 		(in_pos_files yes)
 		(dnp no)
-		(property "Reference" "U1"
+		(property "Reference" "U3"
 			(at 146.05 69.85 0)
 			(show_name no)
@@
 			(project "10001"
 				(path "/74a9143e-df50-4944-bff2-a4302f33bdee/58f0d544-aaa2-42db-8316-207d7dca1f4a"
-					(reference "U1")
+					(reference "U3")
 					(unit 1)
 				)
@@
 		(dnp no)
 		(fields_autoplaced yes)
-		(property "Reference" "#PWR07"
+		(property "Reference" "#PWR014"
 			(at 140.97 107.95 0)
 			(hide yes)
@@
 			(project "10001"
 				(path "/74a9143e-df50-4944-bff2-a4302f33bdee/58f0d544-aaa2-42db-8316-207d7dca1f4a"
-					(reference "#PWR07")
+					(reference "#PWR014")
 					(unit 1)
 				)
@@
 		(dnp no)
 		(fields_autoplaced yes)
-		(property "Reference" "#PWR010"
+		(property "Reference" "#PWR016"
 			(at 160.02 77.47 0)
 			(hide yes)
@@
 			(project "10001"
 				(path "/74a9143e-df50-4944-bff2-a4302f33bdee/58f0d544-aaa2-42db-8316-207d7dca1f4a"
-					(reference "#PWR010")
+					(reference "#PWR016")
 					(unit 1)
 				)
@@
 		(dnp no)
 		(fields_autoplaced yes)
-		(property "Reference" "#PWR08"
+		(property "Reference" "#PWR012"
 			(at 114.3 102.87 0)
 			(hide yes)
@@
 			(project "10001"
 				(path "/74a9143e-df50-4944-bff2-a4302f33bdee/58f0d544-aaa2-42db-8316-207d7dca1f4a"
-					(reference "#PWR08")
+					(reference "#PWR012")
 					(unit 1)
 				)
@@
 		(dnp no)
 		(fields_autoplaced yes)
-		(property "Reference" "#PWR09"
+		(property "Reference" "#PWR013"
 			(at 114.3 130.81 0)
 			(hide yes)
@@
 			(project "10001"
 				(path "/74a9143e-df50-4944-bff2-a4302f33bdee/58f0d544-aaa2-42db-8316-207d7dca1f4a"
-					(reference "#PWR09")
+					(reference "#PWR013")
 					(unit 1)
 				)
@@
 		(dnp no)
 		(fields_autoplaced yes)
-		(property "Reference" "#PWR05"
+		(property "Reference" "#PWR015"
 			(at 142.24 72.39 0)
 			(hide yes)
@@
 			(project "10001"
 				(path "/74a9143e-df50-4944-bff2-a4302f33bdee/58f0d544-aaa2-42db-8316-207d7dca1f4a"
-					(reference "#PWR05")
-					(unit 1)
-				)
+					(reference "#PWR015")
+					(unit 1)
+				)
