File: actuator/10001/micro.kicad_sch (KiCad schematic)
At the start: 3 parts, among them U2 STM32F030R8Tx, U3 CP2102N-Axx-xQFN20, Y1 ECS-2520MV-xxx-xx

Commit message: 10001 schematic work
Parts:
- added C16, C20, C9: 0.1uF, symbol Device:C
- added C17: 4.7uF, symbol Device:C
- added C18: 10nF, symbol Device:C
- added C19: 1uF, symbol Device:C
- added R15: 22, symbol Device:R
Connections:
- net +3.3V: now also C16.1, C17.1, C18.1, C19.1, C20.1, C9.1
- net GND: now also C16.2, C17.2, C18.2, C19.2, C20.2, C9.2
- net at Y1.3 (OUT): now also R15.1
- net at U2.5 (PF0): now also R15.2
- no-connect marks 0 -> 2
Other:
- note added: "PLACE NEAR VDD PINS"
- note added: "PLACE NEAR VDDA PIN"
- company: Jay Maybe -> James May
- moved on the sheet: Y1

Commit message: checkpoint
Parts:
- added C21: 0.1uF, Capacitor_SMD:C_0805_2012Metric, symbol Device:C
- added R16: 10k, Resistor_SMD:R_0805_2012Metric, symbol Device:R
- added TP2: 5019, TestPoint:TestPoint_Keystone_5019_Miniature, symbol Connector:TestPoint
- C1: renamed from C20; footprint (none) -> Capacitor_SMD:C_0805_2012Metric
- C2: renamed from C9; footprint (none) -> Capacitor_SMD:C_0805_2012Metric
- C3: renamed from C16; footprint (none) -> Capacitor_SMD:C_0805_2012Metric
- C4: renamed from C17; footprint (none) -> Capacitor_SMD:C_0805_2012Metric
- C5: renamed from C18; footprint (none) -> Capacitor_SMD:C_0805_2012Metric
- C6: renamed from C19; footprint (none) -> Capacitor_SMD:C_0805_2012Metric
- R1: renamed from R15; footprint (none) -> Resistor_SMD:R_0805_2012Metric
- renumbered U2 to U1, U3 to U2
Connections:
- net GND: now also C21.2, R16.2
- net BOOT0: now reaches U1.60 (BOOT0)
- net BOOT0: now also R16.1
- net at U1.7 (NRST): now also C21.1, TP2.1
