File: actuator/10001/motordriver.kicad_sch (KiCad schematic)
At the start: 1 part, among them J1 Conn_01x02

Commit message: 10001 schematic work
Other:
- company: Jay Maybe -> James May
Changed lines of the file:
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@@
 		(date "2026-07-22")
 		(rev "001")
-		(company "Jay Maybe")
+		(company "James May")
 		(comment 1 "10001-001")
 	)

Commit message: checkpoint
Parts:
- removed J1: Conn_01x02, Connector_PinHeader_2.54mm:PinHeader_1x02_P2.54mm_Vertical, symbol Connector_Generic:Conn_01x02
- added J2: Conn_01x04, symbol Connector_Generic:Conn_01x04
Connections:
- net MOTOR_OUT0: now also J2.2 (Pin_2)
- net MOTOR_OUT1: now also J2.3 (Pin_3)
- new net +3.3V: J2.1 (Pin_1)
- new net GND: J2.4 (Pin_4)
Other:
- note added: "For Rev 001 this is just digital output pins from micro. Intention is to drive an external H bridge."
- note removed: "For Rev 001 this is just pins from the output of the micro."
Changed lines of the file:
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@@
 		(comment 1 "10001-001")
 	)
-	(text "For Rev 001 this is just pins from the output of the micro."
+	(text "For Rev 001 this is just digital output pins from micro.\nIntention is to drive an external H bridge."
 		(exclude_from_sim no)
-		(at 131.064 122.682 0)
+		(at 61.468 90.424 0)
 		(effects
 			(font
@@
 	(wire
 		(pts
+			(xy 115.57 96.52) (xy 115.57 93.98)
+		)
+		(stroke
+			(width 0)
+			(type default)
+		)
+	)
+	(wire
+		(pts
+			(xy 115.57 86.36) (xy 118.11 86.36)
+		)
+		(stroke
+			(width 0)
+			(type default)
+		)
+	)
+	(wire
+		(pts
 			(xy 114.3 88.9) (xy 118.11 88.9)
+		)
+		(stroke
+			(width 0)
+			(type default)
+		)
+	)
+	(wire
+		(pts
+			(xy 115.57 83.82) (xy 115.57 86.36)
+		)
+		(stroke
+			(width 0)
+			(type default)
+		)
+	)
+	(wire
+		(pts
+			(xy 115.57 93.98) (xy 118.11 93.98)
 		)
 		(stroke
@@
 	)
 	(symbol
-		(lib_id "Connector_Generic:Conn_01x02")
+		(lib_id "power:GND")
+		(at 115.57 96.52 0)
+		(unit 1)
+		(body_style 1)
+		(exclude_from_sim no)
+		(in_bom yes)
+		(on_board yes)
+		(in_pos_files yes)
+		(dnp no)
+		(fields_autoplaced yes)
+		(property "Reference" "#PWR033"
+			(at 115.57 102.87 0)
+			(hide yes)
+			(show_name no)
+			(do_not_autoplace no)
+			(effects
+				(font
+					(size 1.27 1.27)
+				)
+			)
+		)
+		(property "Value" "GND"
+			(at 115.57 101.6 0)
+			(show_name no)
+			(do_not_autoplace no)
+			(effects
+				(font
+					(size 1.27 1.27)
+				)
+			)
+		)
+		(property "Footprint" ""
+			(at 115.57 96.52 0)
+			(hide yes)
+			(show_name no)
+			(do_not_autoplace no)
+			(effects
+				(font
+					(size 1.27 1.27)
+				)
+			)
+		)
+		(property "Datasheet" ""
+			(at 115.57 96.52 0)
+			(hide yes)
+			(show_name no)
+			(do_not_autoplace no)
+			(effects
+				(font
+					(size 1.27 1.27)
+				)
+			)
+		)
+		(property "Description" "Power symbol creates a global label with name \"GND\" , ground"
+			(at 115.57 96.52 0)
+			(hide yes)
+			(show_name no)
+			(do_not_autoplace no)
+			(effects
+				(font
+					(size 1.27 1.27)
+				)
+			)
+		)
+		(pin "1"
+		)
+		(instances
+			(project "10001"
+				(path "/74a9143e-df50-4944-bff2-a4302f33bdee/45bb560c-1ac0-46a5-91c2-4b646977388c"
+					(reference "#PWR033")
+					(unit 1)
+				)
+			)
+		)
+	)
+	(symbol
+		(lib_id "power:+3.3V")
+		(at 115.57 83.82 0)
+		(unit 1)
+		(body_style 1)
+		(exclude_from_sim no)
+		(in_bom yes)
+		(on_board yes)
+		(in_pos_files yes)
+		(dnp no)
+		(fields_autoplaced yes)
+		(property "Reference" "#PWR034"
+			(at 115.57 87.63 0)
+			(hide yes)
+			(show_name no)
+			(do_not_autoplace no)
+			(effects
+				(font
+					(size 1.27 1.27)
+				)
+			)
+		)
+		(property "Value" "+3.3V"
+			(at 115.57 78.74 0)
+			(show_name no)
+			(do_not_autoplace no)
+			(effects
+				(font
+					(size 1.27 1.27)
+				)
+			)
+		)
+		(property "Footprint" ""
+			(at 115.57 83.82 0)
+			(hide yes)
+			(show_name no)
+			(do_not_autoplace no)
+			(effects
+				(font
+					(size 1.27 1.27)
+				)
+			)
+		)
+		(property "Datasheet" ""
+			(at 115.57 83.82 0)
+			(hide yes)
+			(show_name no)
+			(do_not_autoplace no)
+			(effects
+				(font
+					(size 1.27 1.27)
+				)
+			)
+		)
+		(property "Description" "Power symbol creates a global label with name \"+3.3V\""
+			(at 115.57 83.82 0)
+			(hide yes)
+			(show_name no)
+			(do_not_autoplace no)
+			(effects
+				(font
+					(size 1.27 1.27)
+				)
+			)
+		)
+		(pin "1"
+		)
+		(instances
+			(project "10001"
+				(path "/74a9143e-df50-4944-bff2-a4302f33bdee/45bb560c-1ac0-46a5-91c2-4b646977388c"
+					(reference "#PWR034")
+					(unit 1)
+				)
+			)
+		)
+	)
+	(symbol
+		(lib_id "Connector_Generic:Conn_01x04")
 		(at 123.19 88.9 0)
 		(unit 1)
@@
 		(dnp no)
 		(fields_autoplaced yes)
-		(property "Reference" "J1"
+		(property "Reference" "J2"
 			(at 125.73 88.8999 0)
 			(show_name no)
@@
 			)
 		)
-		(property "Value" "Conn_01x02"
+		(property "Value" "Conn_01x04"
 			(at 125.73 91.4399 0)
 			(show_name no)
@@
 			)
 		)
-		(property "Footprint" "Connector_PinHeader_2.54mm:PinHeader_1x02_P2.54mm_Vertical"
+		(property "Footprint" ""
 			(at 123.19 88.9 0)
 			(hide yes)
@@
 			)
 		)
-		(property "Description" "Generic connector, single row, 01x02, script generated (kicad-library-utils/schlib/autogen/connector/)"
+		(property "Description" "Generic connector, single row, 01x04, script generated (kicad-library-utils/schlib/autogen/connector/)"
 			(at 123.19 88.9 0)
 			(hide yes)
@@
 			)
 		)
+		(pin "4"
+		)
 		(pin "1"
+		)
+		(pin "3"
 		)
 		(pin "2"
@@
 			(project "10001"
 				(path "/74a9143e-df50-4944-bff2-a4302f33bdee/45bb560c-1ac0-46a5-91c2-4b646977388c"
-					(reference "J1")
+					(reference "J2")
 					(unit 1)
 				)

Commit message: motor driver work
Other:
- note removed: "For Rev 001 this is just digital output pins from micro. Intention is to drive an external H bridge."
Changed lines of the file:
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@@
 		(comment 1 "10001-001")
-	)
-	(text "For Rev 001 this is just digital output pins from micro.\nIntention is to drive an external H bridge."
-		(exclude_from_sim no)
-		(at 61.468 90.424 0)
-		(effects
-			(font
-				(size 1.27 1.27)
-			)
-		)
 	)
 	(wire

Commit message: more motor driver work
Parts:
- added U10, U7, U8, U9: IAUC100N04S6L025, Package_SON:Infineon_PG-TDSON-8_6.15x5.15mm, symbol custom:IAUC100N04S6L025
- added U5, U6: IRS2005S, Package_SO:SOIC-8_3.9x4.9mm_P1.27mm, symbol Driver_FET:IRS2005S
